File: 100 MHz TTL CMOS/100 MHz TTL CMOS.kicad_pcb (KiCad board)
At the start: 2 copper layers, 36 parts, among them IC1 74LS14, IC2 MCP23017_SO, IC3 74HC14, IC4 24LC256, IC5 74HC151, IC6 ULN2003, J1 Conn_01x10_Male, J2 Conn_Coaxial, J3 Conn_01x04_Male, K1 MS05-1A87-75DHR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

Commit message: Updated
Parts:
- K1, K2, K3, K4, K5, K6: value MS05-1A87-75DHR -> UMS05-1A80-75D; footprint Frequenzzaehler:Relay_SPST_StandexMeder_MS_Form1AB -> Relay_THT:Relay_SPST_StandexMeder_MS_Form1AB
Connections:
- net Net-(IC2-Pad1) renamed /BUTTON
- net Net-(IC2-Pad2) renamed /LED
- IC1 pad 10: (no net) -> unconnected-(IC1-Pad10)
- IC1 pad 12: (no net) -> unconnected-(IC1-Pad12)
- IC1 pad 6: (no net) -> unconnected-(IC1-Pad6)
- IC1 pad 8: (no net) -> unconnected-(IC1-Pad8)
- IC2 pad 11: (no net) -> unconnected-(IC2-Pad11)
- IC2 pad 14: (no net) -> unconnected-(IC2-Pad14)
- IC2 pad 19: (no net) -> unconnected-(IC2-Pad19)
- IC2 pad 20: (no net) -> unconnected-(IC2-Pad20)
- IC2 pad 3: (no net) -> unconnected-(IC2-Pad3)
- IC2 pad 4: (no net) -> unconnected-(IC2-Pad4)
- IC2 pad 5: (no net) -> unconnected-(IC2-Pad5)
- IC2 pad 6: (no net) -> unconnected-(IC2-Pad6)
- IC2 pad 7: (no net) -> unconnected-(IC2-Pad7)
- IC2 pad 8: (no net) -> unconnected-(IC2-Pad8)
- IC5 pad 6: (no net) -> unconnected-(IC5-Pad6)
- IC6 pad 10: (no net) -> unconnected-(IC6-Pad10)
- J1 pad 4: (no net) -> unconnected-(J1-Pad4)
- K1 pad 3: Net-(IC6-Pad16) -> VCC
- K2 pad 3: Net-(IC6-Pad15) -> VCC
- K3 pad 3: Net-(IC6-Pad13) -> VCC
- K4 pad 3: Net-(IC6-Pad14) -> VCC
- K5 pad 3: Net-(IC6-Pad12) -> VCC
- K6 pad 3: Net-(IC6-Pad11) -> VCC
- SW1 pad 4: (no net) -> unconnected-(SW1-Pad4)
- SW1 pad 5: (no net) -> unconnected-(SW1-Pad5)
- SW2 pad 4: (no net) -> unconnected-(SW2-Pad4)
- SW2 pad 5: (no net) -> unconnected-(SW2-Pad5)
Routing:
- net GND: track 9.34 -> 5.08 mm
Other:
- board outline added: 158.1 x 50.8 mm
- net class Default removed
- net class Versorgung removed
