File: Hauptplatine/Grundplatine.kicad_sch (KiCad schematic)
At the start: 8 parts, among them IC12 Arduino_Nano_v2.x, IC26 74HC00

Commit message: Short break in reset
Connections:
- net VCC: no longer IC12.28 (~{RESET}), IC12.3 (~{RESET})
- no-connect marks 21 -> 23
Changed lines of the file:
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@@
   (junction (at 212.09 69.85) (diameter 0) (color 0 0 0 0)
   )
-  (junction (at 110.49 44.45) (diameter 0) (color 0 0 0 0)
-  )
   (junction (at 92.71 189.23) (diameter 0) (color 0 0 0 0)
   )
@@
   )
   (junction (at 97.79 113.03) (diameter 0) (color 0 0 0 0)
-  )
-  (junction (at 110.49 41.91) (diameter 0) (color 0 0 0 0)
   )
   (junction (at 97.79 148.59) (diameter 0) (color 0 0 0 0)
@@
   (no_connect (at 77.47 156.21))
   (no_connect (at 148.59 31.75))
+  (no_connect (at 140.97 44.45))
+  (no_connect (at 140.97 41.91))
   (no_connect (at 166.37 46.99))
   (no_connect (at 166.37 64.77))
@@
     (stroke (width 0) (type default) (color 0 0 0 0))
   )
-  (wire (pts (xy 140.97 41.91) (xy 110.49 41.91))
-    (stroke (width 0) (type default) (color 0 0 0 0))
-  )
   (wire (pts (xy 110.49 181.61) (xy 110.49 146.05))
     (stroke (width 0) (type default) (color 0 0 0 0))
@@
     (stroke (width 0) (type default) (color 0 0 0 0))
   )
-  (wire (pts (xy 110.49 41.91) (xy 110.49 12.7))
+  (wire (pts (xy 110.49 12.7) (xy 110.49 74.93))
     (stroke (width 0) (type default) (color 0 0 0 0))
   )
@@
     (stroke (width 0) (type default) (color 0 0 0 0))
   )
-  (wire (pts (xy 110.49 44.45) (xy 110.49 74.93))
-    (stroke (width 0) (type default) (color 0 0 0 0))
-  )
   (wire (pts (xy 166.37 69.85) (xy 212.09 69.85))
     (stroke (width 0) (type default) (color 0 0 0 0))
@@
     (stroke (width 0) (type default) (color 0 0 0 0))
   )
-  (wire (pts (xy 110.49 41.91) (xy 110.49 44.45))
-    (stroke (width 0) (type default) (color 0 0 0 0))
-  )
   (wire (pts (xy 77.47 163.83) (xy 92.71 163.83))
     (stroke (width 0) (type default) (color 0 0 0 0))
@@
   )
   (wire (pts (xy 77.47 74.93) (xy 110.49 74.93))
-    (stroke (width 0) (type default) (color 0 0 0 0))
-  )
-  (wire (pts (xy 140.97 44.45) (xy 110.49 44.45))
     (stroke (width 0) (type default) (color 0 0 0 0))
   )
@@
       (effects (font (size 1.27 1.27)) hide)
     )
+    (pin "1")
+    (pin "2")
+    (pin "3")
     (pin "4")
     (pin "5")
     (pin "6")
-  )
-  (symbol (lib_id "power:GND") (at 92.71 196.85 0)
+    (pin "10")
+    (pin "8")
+    (pin "9")
+    (pin "11")
+    (pin "12")
+    (pin "13")
+    (pin "14")
+    (pin "7")
+  )
+  (symbol (lib_id "power:GND") (at 92.71 196.85 0) (unit 1)
     (in_bom yes) (on_board yes)
     (property "Reference" "#PWR0108" (id 0) (at 92.71 203.2 0)
@@
     (pin "1")
   )
-  (symbol (lib_id "power:GND") (at 153.67 97.79 0)
+  (symbol (lib_id "power:GND") (at 153.67 97.79 0) (unit 1)
     (in_bom yes) (on_board yes)
     (property "Reference" "#PWR0109" (id 0) (at 153.67 104.14 0)
@@
     (pin "1")
   )
-  (symbol (lib_id "power:VCC") (at 156.21 7.62 0)
+  (symbol (lib_id "power:VCC") (at 156.21 7.62 0) (unit 1)
     (in_bom yes) (on_board yes)
     (property "Reference" "#PWR0110" (id 0) (at 156.21 11.43 0)

Commit message: Update
Parts:
- added C1: 100n, Capacitor_THT:C_Rect_L10.0mm_W4.0mm_P7.50mm_FKS3_FKP3, symbol Hauptplatine-rescue:C-EUC0603-Zähler-eagle-import
- added D2, D3: 1N4148, Diode_THT:D_DO-35_SOD27_P7.62mm_Horizontal, symbol Device:D
- added R11: 1k, Resistor_THT:R_Axial_DIN0204_L3.6mm_D1.6mm_P1.90mm_Vertical, symbol Hauptplatine-rescue:R-EU_M0805-Grundplatine-eagle-import
- added R12: 10k, Resistor_THT:R_Axial_DIN0204_L3.6mm_D1.6mm_P1.90mm_Vertical, symbol Hauptplatine-rescue:R-EU_M0805-Grundplatine-eagle-import
Connections:
- net 0.5HZ: now also D3.1 (K); no longer IC12.10 (D7)
- net DONE: now also D2.1 (K); no longer IC12.9 (D6)
- net GND: now also C1.2
- net VCC: no longer IC12.30 (VIN)
- net at IC12.17 (3V3): now also R11.2, R12.2
- new net: D3.2 (A), IC12.10 (D7), R11.1
- new net: D2.2 (A), IC12.9 (D6), R12.1
- new net VDD: C1.1, IC12.30 (VIN)
- no-connect marks 23 -> 22
Other:
- moved on the sheet: IC26B
