File: Hauptplatine/Hauptplatine.kicad_pcb (KiCad board)
At the start: 2 copper layers, 179.7 x 194.9 mm, 47 parts, among them IC1 74HC4040, IC10 74HC02, IC12 Arduino_Nano_v2.x, IC2 74HC4040, IC20 74HC04, IC21 74HC390, IC22 74HC390, IC23 74HC390, IC24 74HC390, IC25 74HC107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

Commit message: Update
Parts:
- added C1: 100n, Capacitor_THT:C_Rect_L10.0mm_W4.0mm_P7.50mm_FKS3_FKP3, F.Cu at (153.7, 11.4)
- added D2: 1N4148, Diode_THT:D_DO-35_SOD27_P7.62mm_Horizontal, F.Cu at (134.2, 34.9)
- added D3: 1N4148, Diode_THT:D_DO-35_SOD27_P7.62mm_Horizontal, F.Cu at (134.1, 24.8)
- added R11: 1k, Resistor_THT:R_Axial_DIN0204_L3.6mm_D1.6mm_P1.90mm_Vertical, F.Cu at (145.2, 24.8)
- added R12: 10k, Resistor_THT:R_Axial_DIN0204_L3.6mm_D1.6mm_P1.90mm_Vertical, F.Cu at (145.2, 34.9)
Connections:
- C14 pad 1: Net-(C14-Pad1) -> VDD
- C30 pad 1: Net-(C14-Pad1) -> VDD
- D1 pad 1: Net-(C14-Pad1) -> VDD
- IC12 pad 10: 0.5HZ -> Net-(IC12-Pad10)
- IC12 pad 17: unconnected-(IC12-Pad17) -> Net-(IC12-Pad17)
- IC12 pad 30: VCC -> VDD
- IC12 pad 9: DONE -> Net-(IC12-Pad9)
- IC20 pad 1: GND -> Net-(IC8-Pad3)
- IC20 pad 2: unconnected-(IC20-Pad2) -> DONE
- IC8 pad 3: DONE -> Net-(IC8-Pad3)
- U1 pad 1: Net-(C14-Pad1) -> VDD
Routing:
- net Net-(IC8-Pad3): track 0.00 -> 150.5 mm, vias 0 -> 3
- net VDD: track 0.00 -> 130.4 mm
- net DONE: track 166.4 -> 43.1 mm
- net Net-(IC12-Pad17): track 0.00 -> 66.2 mm, vias 0 -> 1
- net 0.5HZ: track 217.9 -> 169.5 mm, vias 3 -> 2
- net Net-(C14-Pad1): track 45.1 -> 0.00 mm
- net Net-(IC12-Pad10): track 0.00 -> 40.8 mm, vias 0 -> 1
- net Net-(IC12-Pad9): track 0.00 -> 34.0 mm
- net VCC: track 1871.1 -> 1861.4 mm
- net RESET_FF: track 87.5 -> 89.0 mm
- net SDA: track 312.0 -> 311.2 mm
