File: Hauptplatine/Netzteil.kicad_sch (KiCad schematic)
At the start: 8 parts, among them J1 Screw_Terminal_01x03, U1 L7805

Commit message: Update
Connections:
- net VDD: now reaches C14.1, C30.1, D1.1 (+), U1.1 (IN)
Changed lines of the file:
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@@
+    (stroke (width 0) (type default) (color 0 0 0 0))
+  )
+  (wire (pts (xy 119.38 25.4) (xy 119.38 33.02))
     (stroke (width 0) (type default) (color 0 0 0 0))
   )
@@
       (effects (font (size 1.27 1.27)) hide)
     )
+    (pin "1")
+  )
+  (symbol (lib_id "power:VDD") (at 119.38 25.4 0) (unit 1)
+    (in_bom yes) (on_board yes) (fields_autoplaced)
+    (property "Reference" "#PWR02" (id 0) (at 119.38 29.21 0)
+      (effects (font (size 1.27 1.27)) hide)
+    )
+    (property "Value" "VDD" (id 1) (at 119.38 20.32 0))
+    (property "Footprint" "" (id 2) (at 119.38 25.4 0)
+      (effects (font (size 1.27 1.27)) hide)
+    )
+    (property "Datasheet" "" (id 3) (at 119.38 25.4 0)
+      (effects (font (size 1.27 1.27)) hide)
+    )
