File: Hauptplatine/Taktgenerator.kicad_sch (KiCad schematic)
At the start: 10 parts, among them IC20 74HC04, IC21 74HC390, IC22 74HC390, IC23 74HC390, IC24 74HC390, IC25 74HC107, IC26 74HC00, IC27 XO-14, J3 Conn_Coaxial

Commit message: Update
Parts:
- removed unit 1 of IC20
Connections:
- no-connect marks 21 -> 20
Changed lines of the file:
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@@
   (junction (at 137.16 73.66) (diameter 0) (color 0 0 0 0)
-  )
-  (junction (at 246.38 177.8) (diameter 0) (color 0 0 0 0)
   )
   (junction (at 100.33 191.77) (diameter 0) (color 0 0 0 0)
@@
   (no_connect (at 205.74 68.58))
   (no_connect (at 205.74 71.12))
-  (no_connect (at 270.51 157.48))
   (no_connect (at 243.84 43.18))
   (no_connect (at 167.64 43.18))
@@
     (stroke (width 0) (type default) (color 0 0 0 0))
   )
-  (wire (pts (xy 246.38 157.48) (xy 246.38 177.8))
-    (stroke (width 0) (type default) (color 0 0 0 0))
-  )
   (wire (pts (xy 208.28 33.02) (xy 177.8 33.02))
     (stroke (width 0) (type default) (color 0 0 0 0))
@@
   )
   (wire (pts (xy 139.7 55.88) (xy 139.7 68.58))
-    (stroke (width 0) (type default) (color 0 0 0 0))
-  )
-  (wire (pts (xy 250.19 157.48) (xy 246.38 157.48))
     (stroke (width 0) (type default) (color 0 0 0 0))
   )
@@
       (effects (font (size 1.27 1.27)) hide)
     )
-    (pin "1")
-    (pin "2")
-    (pin "3")
-    (pin "4")
-    (pin "5")
-    (pin "6")
-    (pin "8")
-    (pin "9")
-    (pin "10")
-    (pin "11")
-    (pin "12")
-    (pin "13")
-    (pin "14")
-    (pin "7")
-  )
-  (symbol (lib_id "Hauptplatine-rescue:7404D-Taktgenerator-eagle-import") (at 260.35 157.48 0) (unit 1)
-    (in_bom yes) (on_board yes)
-    (property "Reference" "IC20" (id 0) (at 256.54 165.1 0)
-      (effects (font (size 1.4986 1.4986)) (justify left bottom))
-    )
-    (property "Value" "74HC04" (id 1) (at 262.89 162.56 0)
-      (effects (font (size 1.4986 1.4986)) (justify left bottom) hide)
-    )
-    (property "Footprint" "Package_DIP:DIP-14_W7.62mm_LongPads" (id 2) (at 260.35 157.48 0)
-      (effects (font (size 1.27 1.27)) hide)
-    )
-    (property "Datasheet" "https://cdn-reichelt.de/documents/datenblatt/A240/74HC04%23STM.pdf" (id 3) (at 260.35 157.48 0)
-      (effects (font (size 1.27 1.27)) hide)
-    )
