File: Hauptplatine/Zähler.kicad_sch (KiCad schematic)
At the start: 24 parts, among them IC1 74HC4040, IC10 74HC02, IC2 74HC4040, IC25 74HC107, IC26 74HC00, IC3 74HC4040, IC4 MCP23017SO, IC5 MCP23017SO, IC6 74HC107, IC7 74HC151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

Commit message: Update
Parts:
- added IC20: 74HC04, Package_DIP:DIP-14_W7.62mm_LongPads, symbol Hauptplatine-rescue:7404D-Taktgenerator-eagle-import
Connections:
- net DONE: now also IC20.2 (O); no longer IC8.3 (Q)
- new net: IC20.1 (I), IC8.3 (Q)
Changed lines of the file:
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@@
+    (stroke (width 0) (type default) (color 0 0 0 0))
+  )
+  (wire (pts (xy 130.81 137.16) (xy 143.51 137.16))
     (stroke (width 0) (type default) (color 0 0 0 0))
   )
@@
     (stroke (width 0) (type default) (color 0 0 0 0))
   )
-  (wire (pts (xy 173.99 137.16) (xy 158.75 137.16))
+  (wire (pts (xy 173.99 137.16) (xy 163.83 137.16))
     (stroke (width 0) (type default) (color 0 0 0 0))
   )
@@
     )
   )
-  (global_label "DONE" (shape output) (at 158.75 137.16 180) (fields_autoplaced)
+  (global_label "DONE" (shape output) (at 130.81 137.16 180) (fields_autoplaced)
     (effects (font (size 1.27 1.27)) (justify right))
-    (property "Intersheet References" "${INTERSHEET_REFS}" (id 0) (at 0 0 0)
+    (property "Intersheet References" "${INTERSHEET_REFS}" (id 0) (at -27.94 0 0)
       (effects (font (size 1.27 1.27)) hide)
     )
@@
     (pin "1")
   )
+  (symbol (lib_id "Hauptplatine-rescue:7404D-Taktgenerator-eagle-import") (at 153.67 137.16 180) (unit 1)
+    (in_bom yes) (on_board yes)
+    (property "Reference" "IC20" (id 0) (at 157.48 129.54 0)
+      (effects (font (size 1.4986 1.4986)) (justify left bottom))
+    )
+    (property "Value" "74HC04" (id 1) (at 151.13 132.08 0)
+      (effects (font (size 1.4986 1.4986)) (justify left bottom) hide)
+    )
+    (property "Footprint" "Package_DIP:DIP-14_W7.62mm_LongPads" (id 2) (at 153.67 137.16 0)
+      (effects (font (size 1.27 1.27)) hide)
+    )
+    (property "Datasheet" "https://cdn-reichelt.de/documents/datenblatt/A240/74HC04%23STM.pdf" (id 3) (at 153.67 137.16 0)
+      (effects (font (size 1.27 1.27)) hide)
+    )
+    (pin "1")
+    (pin "2")
+    (pin "3")
+    (pin "4")
+    (pin "5")
+    (pin "6")
+    (pin "8")
+    (pin "9")
+    (pin "10")
+    (pin "11")
+    (pin "12")
+    (pin "13")
+    (pin "14")
+    (pin "7")
+  )
   (symbol (lib_id "power:GND") (at 276.86 128.27 0) (unit 1)
